File: DriveSystems/DriveSystems.kicad_sch (KiCad schematic)
At the start: 30 parts, among them J1 Raspberry_Pi_4, J2 RJ45, M1 Motor_Servo, M2 Motor_Servo, SW1 SW_Rotary_1x2_MP, U1 RoboClaw Motor Controller, U2 5304 Gear Motor, U3 5VDC 5A UBC-C PSU, U4 24V 5V10A DCDC Stepdown, U5 RoboClaw VClamp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

Commit message: Update DriveSystems.kicad_sch
Parts:
- added A1: Arduino_Leonardo, Module:Arduino_UNO_R3, symbol MCU_Module:Arduino_Leonardo
Connections:
- net at U1. (EN1_A): now also R6.2
- net at F3.2, F4.2, U4.3 (5Vout): now also A1.8 (VIN)
- net at M1.3 (-), M2.3 (-), U4.4 (GND): now also A1.7 (GND)
Changed lines of the file:
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@@
 		(color 0 0 0 0)
 	)
+	(junction
+		(at 87.63 162.56)
+		(diameter 0)
+		(color 0 0 0 0)
+	)
+	(junction
+		(at 85.09 165.1)
+		(diameter 0)
+		(color 0 0 0 0)
+	)
 	(wire
 		(pts
@@
 	(wire
 		(pts
+			(xy 13.97 162.56) (xy 13.97 185.42)
+		)
+		(stroke
+			(width 0)
+			(type default)
+		)
+	)
+	(wire
+		(pts
 			(xy 99.06 125.73) (xy 143.51 125.73)
 		)
@@
 	(wire
 		(pts
+			(xy 13.97 162.56) (xy 87.63 162.56)
+		)
+		(stroke
+			(width 0)
+			(type default)
+		)
+	)
+	(wire
+		(pts
 			(xy 205.74 85.09) (xy 214.63 85.09)
 		)
@@
 	(wire
 		(pts
+			(xy 13.97 185.42) (xy 19.05 185.42)
+		)
+		(stroke
+			(width 0)
+			(type default)
+		)
+	)
+	(wire
+		(pts
 			(xy 181.61 104.14) (xy 181.61 157.48)
 		)
@@
 	(wire
 		(pts
+			(xy 85.09 165.1) (xy 73.66 165.1)
+		)
+		(stroke
+			(width 0)
+			(type default)
+		)
+	)
+	(wire
+		(pts
 			(xy 69.85 147.32) (xy 69.85 160.02)
 		)
@@
 	(wire
 		(pts
+			(xy 73.66 180.34) (xy 72.39 180.34)
+		)
+		(stroke
+			(width 0)
+			(type default)
+		)
+	)
+	(wire
+		(pts
 			(xy 233.68 116.84) (xy 275.59 116.84)
 		)
@@
 	(wire
 		(pts
+			(xy 73.66 165.1) (xy 73.66 180.34)
+		)
+		(stroke
+			(width 0)
+			(type default)
+		)
+	)
+	(wire
+		(pts
 			(xy 240.03 139.7) (xy 246.38 139.7)
 		)
@@
 		)
 	)
+	(label "Ardunio connections not pictured (contact John)"
+		(at 25.4 167.64 0)
+		(effects
+			(font
+				(size 1.27 1.27)
+			)
+			(justify left bottom)
+		)
+	)
+	(label "Power to Arduino delivered through DC Jack"
+		(at 25.4 165.1 0)
+		(effects
+			(font
+				(size 1.27 1.27)
+			)
+			(justify left bottom)
+		)
+	)
 	(symbol
 		(lib_id "Connector:Raspberry_Pi_4")
@@
 					(unit 1)
 				)
+			)
+		)
+	)
+	(symbol
+		(lib_id "MCU_Module:Arduino_Leonardo")
+		(at 44.45 182.88 90)
+		(unit 1)
+		(exclude_from_sim no)
+		(in_bom yes)
+		(on_board yes)
+		(dnp no)
+		(property "Reference" "A1"
+			(at 51.308 178.308 90)
+			(effects
+				(font
+					(size 1.27 1.27)
+				)
+			)
+		)
+		(property "Value" "Arduino_Leonardo"
+			(at 49.022 182.626 90)
+			(effects
+				(font
+					(size 1.27 1.27)
+				)
+			)
+		)
+		(property "Footprint" "Module:Arduino_UNO_R3"
+			(at 44.45 182.88 0)
+			(effects
+				(font
+					(size 1.27 1.27)
+					(italic yes)
+				)
+				(hide yes)
+			)
+		)
+		(property "Datasheet" "https://www.arduino.cc/en/Main/ArduinoBoardLeonardo"
+			(at 44.45 182.88 0)
+			(effects
+				(font
+					(size 1.27 1.27)
+				)
+				(hide yes)
+			)
+		)
+		(property "Description" "Arduino LEONARDO Microcontroller Module"
+			(at 44.45 182.88 0)
+			(effects
+				(font
+					(size 1.27 1.27)
+				)
+				(hide yes)
+			)
+		)
+		(pin "15"
+		)
+		(pin "16"
+		)
+		(pin "17"
+		)
+		(pin "18"
+		)
+		(pin "19"
+		)
+		(pin "20"
+		)
+		(pin "21"
+		)
+		(pin "22"
+		)
+		(pin "23"
+		)
+		(pin "24"
+		)
+		(pin "25"
+		)
+		(pin "26"
+		)
+		(pin "27"
+		)
+		(pin "28"
+		)
+		(pin "3"
+		)
+		(pin "2"
+		)
+		(pin "30"
+		)
+		(pin "9"
+		)
+		(pin "10"
+		)
+		(pin "11"
+		)
+		(pin "12"
+		)
+		(pin "13"
+		)
+		(pin "14"
+		)
+		(pin "1"
+		)
+		(pin "8"
+		)
+		(pin "29"
+		)
+		(pin "6"
+		)
+		(pin "4"
+		)
+		(pin "7"
+		)
+		(pin "5"
+		)
+		(pin "31"
+		)
+		(pin "32"
+		)
+		(instances
+			(project ""
+				(path "/09f307af-601f-4645-b594-daaafb49fd2a"
+					(reference "A1")
+					(unit 1)
+				)

Commit message: Update DriveSystems.kicad_sch
Connections:
- net at U1. (EN1_A): now also R6.2
Changed lines of the file:
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@@
 	)
 	(label "Ardunio connections not pictured (contact John)"
-		(at 25.4 167.64 0)
+		(at 22.86 167.64 0)
 		(effects
 			(font

Commit message: Update DriveSystems.kicad_sch
Connections:
- net at J1.13 (GPIO27/SDIO_DAT3): now also J2.7
- net at J1.37 (GPIO26/SDIO_DAT2): now also J2.6
- net at U1. (EN1_A): now also R6.2
- net at A1.10 (A1): now also J2.7
- net at A1.9 (A0): now also J2.6
Changed lines of the file:
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@@
+	(wire
+		(pts
+			(xy 97.79 121.92) (xy 80.01 121.92)
+		)
+		(stroke
+			(width 0)
+			(type default)
+		)
+	)
 	(wire
 		(pts
@@
 	(wire
 		(pts
+			(xy 99.06 90.17) (xy 97.79 90.17)
+		)
+		(stroke
+			(width 0)
+			(type default)
+		)
+	)
+	(wire
+		(pts
 			(xy 15.24 57.15) (xy 26.67 57.15)
 		)
@@
 	(wire
 		(pts
+			(xy 99.06 123.19) (xy 82.55 123.19)
+		)
+		(stroke
+			(width 0)
+			(type default)
+		)
+	)
+	(wire
+		(pts
 			(xy 205.74 85.09) (xy 214.63 85.09)
 		)
@@
 	(wire
 		(pts
+			(xy 82.55 154.94) (xy 46.99 154.94)
+		)
+		(stroke
+			(width 0)
+			(type default)
+		)
+	)
+	(wire
+		(pts
 			(xy 172.72 90.17) (xy 172.72 118.11)
 		)
@@
 	(wire
 		(pts
+			(xy 46.99 154.94) (xy 46.99 170.18)
+		)
+		(stroke
+			(width 0)
+			(type default)
+		)
+	)
+	(wire
+		(pts
 			(xy 173.99 97.79) (xy 173.99 127)
+		)
+		(stroke
+			(width 0)
+			(type default)
+		)
+	)
+	(wire
+		(pts
+			(xy 80.01 121.92) (xy 80.01 127)
 		)
 		(stroke
@@
 	(wire
 		(pts
+			(xy 99.06 92.71) (xy 99.06 123.19)
+		)
+		(stroke
+			(width 0)
+			(type default)
+		)
+	)
+	(wire
+		(pts
 			(xy 226.06 102.87) (xy 228.6 102.87)
 		)
@@
 	(wire
 		(pts
+			(xy 80.01 153.67) (xy 44.45 153.67)
+		)
+		(stroke
+			(width 0)
+			(type default)
+		)
+	)
+	(wire
+		(pts
 			(xy 100.33 137.16) (xy 184.15 137.16)
 		)
@@
 	(wire
 		(pts
+			(xy 82.55 147.32) (xy 82.55 154.94)
+		)
+		(stroke
+			(width 0)
+			(type default)
+		)
+	)
+	(wire
+		(pts
 			(xy 233.68 109.22) (xy 233.68 116.84)
 		)
@@
 	(wire
 		(pts
+			(xy 44.45 153.67) (xy 44.45 170.18)
+		)
+		(stroke
+			(width 0)
+			(type default)
+		)
+	)
+	(wire
+		(pts
 			(xy 50.8 125.73) (xy 50.8 130.81)
 		)
@@
 	(wire
 		(pts
+			(xy 80.01 147.32) (xy 80.01 153.67)
+		)
+		(stroke
+			(width 0)
+			(type default)
+		)
+	)
+	(wire
+		(pts
 			(xy 85.09 165.1) (xy 73.66 165.1)
 		)
@@
 	(wire
 		(pts
+			(xy 82.55 123.19) (xy 82.55 127)
+		)
+		(stroke
+			(width 0)
+			(type default)
+		)
+	)
+	(wire
+		(pts
 			(xy 26.67 123.19) (xy 26.67 121.92)
 		)
@@
 		)
 	)
+	(wire
+		(pts
+			(xy 97.79 90.17) (xy 97.79 121.92)
+		)
+		(stroke
+			(width 0)
+			(type default)
+		)
+	)
 	(label "Ardunio connections not pictured (contact John)"
-		(at 22.86 167.64 0)
+		(at 17.78 161.29 0)
 		(effects
 			(font
@@
 	)
 	(label "Power to Arduino delivered through DC Jack"
-		(at 25.4 165.1 0)
+		(at 20.32 158.75 0)
 		(effects
 			(font

Commit message: Update DriveSystems.kicad_sch
Connections:
- net at U1. (EN1_A): now also R6.2
Changed lines of the file:
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@@
 		)
 	)
-	(label "Ardunio connections not pictured (contact John)"
+	(label "Ardunio connections not pictured (contact Jon)"
 		(at 17.78 161.29 0)
 		(effects

Commit message: As built
Connections:
- net at U1. (EN1_A): now also R6.2
- net at J2.3: now also U1.S4 (Brake); no longer U1.S5 (Brake)
- new net: J2.8, R6.1, U1.S5 (E-STOP)

Commit message: Final Cleanup
Connections:
- net at J1.23 (SCLK_SPI0/GPIO11): no longer J2.3
- net 0V: now reaches U1. (EN1_A)
- net 0V: now also U1.4 (Vin-), U2.4 (GND), U3.2 (GND), U4.2 (GND), U5.3 (GND), U5.4 (GND), U7.2 (GND)
- net +5V: now reaches U1. (EN1_A), U2.3 (VCC), U5.2 (+5V)
- net at U1.S4 (Disabled): no longer J2.3
- net +24V: now reaches F1.2, F2.1, F5.1, F6.2
- net +24V: now also CB1.2
Other:
- note removed: "12AWG Wire"
- moved on the sheet: F5, F6, U5

Commit message: NO Switch
Parts:
- removed R5: 10k, symbol Device:R
Connections:
- net at J1.36 (GPIO16/SPI1_~{CE2}): no longer SW1.2
Other:
- moved on the sheet: R1, R2, R3, R4

Commit message: Update DriveSystems.kicad_sch
Connections:
- net at J1.40 (GPIO21/SPI1_SCLK/PCM_DOUT): now also Estop1.1, J2.8
Changed lines of the file:
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@@
+	)
+	(junction
+		(at 50.8 125.73)
+		(diameter 0)
+		(color 0 0 0 0)
 	)
 	(junction
@@
 	(wire
 		(pts
+			(xy 50.8 111.76) (xy 87.63 111.76)
+		)
+		(stroke
+			(width 0)
+			(type default)
+			(color 255 0 0 1)
+		)
+	)
+	(wire
+		(pts
 			(xy 59.69 69.85) (xy 99.06 69.85)
 		)
@@
 	(wire
 		(pts
+			(xy 87.63 111.76) (xy 87.63 74.93)
+		)
+		(stroke
+			(width 0)
+			(type default)
+			(color 255 0 0 1)
+		)
+	)
+	(wire
+		(pts
 			(xy 13.97 185.42) (xy 19.05 185.42)
 		)
@@
 		(pts
 			(xy 193.04 114.3) (xy 194.31 114.3)
+		)
+		(stroke
+			(width 0)
+			(type default)
+			(color 255 0 0 1)
+		)
+	)
+	(wire
+		(pts
+			(xy 50.8 125.73) (xy 50.8 111.76)
 		)
 		(stroke
@@
 	(wire
 		(pts
+			(xy 87.63 74.93) (xy 99.06 74.93)
+		)
+		(stroke
+			(width 0)
+			(type default)
+			(color 255 0 0 1)
+		)
+	)
+	(wire
+		(pts
 			(xy 43.18 69.85) (xy 43.18 106.68)
 		)
@@
 		)
 		(stroke
-			(width 0)
-			(type default)
-		)
-	)
-	(wire
-		(pts
-			(xy 120.65 93.98) (xy 120.65 90.17)
-		)
-		(stroke
